Commit message: added inertia and collision

File: src/my_robot_description/urdf/common_properties.xacro (robot description, xacro)
@@ -7,3 +7,33 @@
         <color rgba="0.5 0.5 0.5 1" />
     </material>
+    <xacro:macro name="box_inertia" params="m l w h xyz rpy" >
+        <inertial>
+            <origin xyz="${xyz}"  rpy="${rpy}" />
+            <mass value="${m}" />
+            <inertia ixx="${(m/12) * (h*h + l*l)}" ixy="0" ixz="0"
+                     iyy="${(m/12) * (w*w + l*l)}" iyz="0"
+                     izz="${(m/12) * (w*w + h*h)}" >
+            </inertia>
+        </inertial>
+    </xacro:macro>
+    <xacro:macro name="cylinder_inertia" params="m r h xyz rpy" >
+        <inertial>
+            <origin xyz="${xyz}"  rpy="${rpy}" />
+            <mass value="${m}" />
+            <inertia ixx="${(m/12) * (3*r*r + h*h)}" ixy="0" ixz="0"
+                     iyy="${(m/12) * (3*(r*r) + h*h)}" iyz="0"
+                     izz="${(m/2) * (r*r)}" >
+            </inertia>
+        </inertial>
+    </xacro:macro>
+    <xacro:macro name="sphere_inertia" params="m r xyz rpy" >
+        <inertial>
+            <origin xyz="${xyz}"  rpy="${rpy}" />
+            <mass value="${m}" />
+            <inertia ixx="${(2/5)* m * r*r}" ixy="0" ixz="0"
+                     iyy="${(2/5) * m * r*r}" iyz="0"
+                     izz="${(2/5) * m * r*r}"   >
+            </inertia>
+        </inertial>
+    </xacro:macro>
 </robot>

File: src/my_robot_description/urdf/mobile_base.xacro (robot description, xacro)
@@ -14,4 +14,12 @@
             <material name="blue" />
         </visual>
+        <collision>
+            <geometry>
+                <box size="${base_length} ${base_width} ${base_hight}" />
+            </geometry>
+            <origin xyz="0 0 ${base_hight / 2.0}" rpy="0 0 0" />
+        </collision>
+        <xacro:box_inertia m="5.0" l="${base_length}" w="${base_width}" h="${base_hight}"
+                           xyz="0 0 ${base_hight / 2.0}" rpy="0 0 0" />
     </link>
     <xacro:macro name="wheel_link" params="prefix">
@@ -24,4 +32,12 @@
                 <material name="grey" />
             </visual>
+            <collision>
+                <geometry>
+                    <cylinder radius="${wheel_radius}" length="${wheel_length}" />
+                </geometry>
+                <origin xyz="0 0 0" rpy="${pi / 2.0} 0 0" />
+            </collision>
+            <xacro:cylinder_inertia m="1.0" r="${wheel_radius}" h="${wheel_length}"
+                                    xyz="0 0 0" rpy="${pi / 2.0} 0 0" />
         </link>
     </xacro:macro>
@@ -36,4 +52,12 @@
             <material name="grey" />
         </visual>
+        <collision>
+            <geometry>
+                <sphere radius="${wheel_radius / 2.0}" />
+            </geometry>
+            <origin xyz="0 0 0" rpy="0 0 0" />
+        </collision>
+        <xacro:sphere_inertia m="0.5" r="${wheel_radius / 2.0}"
+                            xyz="0 0 0" rpy="0 0 0" />
     </link>
     <link name="base_footprint">

Commit message: course project

File: src/my_robot_description/urdf/common_properties.xacro (robot description, xacro)
@@ -6,4 +6,10 @@
     <material name="grey">
         <color rgba="0.5 0.5 0.5 1" />
+    </material>
+    <material name="orange">
+        <color rgba="1 0.65 0 1" />
+    </material>
+    <material name="yellow">
+        <color rgba="1 1 0 1" />
     </material>
     <xacro:macro name="box_inertia" params="m l w h xyz rpy" >

File: src/my_robot_description/urdf/my_robot.urdf.xacro (robot description, xacro)
@@ -5,3 +5,10 @@
     <xacro:include filename="camera.xacro" />
     <xacro:include filename="mobile_base_gazebo.xacro" />
+    <xacro:include filename="arm.xacro" />
+    <xacro:include filename="arm_gazebo.xacro" />
+    <joint name="base_arm_joint" type="fixed">
+        <parent link="base_link" />
+        <child link="arm_base_link" />
+        <origin xyz="${base_length / 3.0} 0 ${base_hight}" rpy="0 0 ${pi / 2.0}" />
+    </joint>
 </robot>
